Commit message: mejorado el mira_custom.urdf

File: src/my_mira_description/urdf/mira_custom.urdf (robot description, URDF)
Before this commit: robot mira, 7 links, 6 joints
Joints:
- joint pitch_joint: origin xyz=0 0 0.105 rpy=0 0 0 -> xyz=0 0 0 rpy=0 0 0; parent base_link -> roll_M1_link
- joint yaw_joint: origin xyz=0 0 0.105 rpy=0 0 0 -> xyz=0 0 0 rpy=0 0 0; parent base_link -> pitch_M2_link
