Commit message: extras en scripts para el control de gurdy

File: src/my_gurdy_description/urdf/gurdy_v2.urdf (robot description, URDF)
Before this commit: robot gurdy, 11 links, 10 joints
Links:
- added link upperleg_M1_yaw_link, mass 0.01; collision cylinder length=0.06 radius=0.0025; visual cylinder length=0.008 radius=0.008
- added link upperleg_M2_yaw_link, mass 0.01; collision cylinder length=0.06 radius=0.0025; visual cylinder length=0.008 radius=0.008
- added link upperleg_M3_yaw_link, mass 0.01; collision cylinder length=0.06 radius=0.0025; visual cylinder length=0.008 radius=0.008
Joints:
- added joint head_upperlegM1_yaw_joint: type revolute, parent head_link, child upperleg_M1_yaw_link, origin xyz=-0.02165 -0.0125 -0.008 rpy=0 0 0, axis 0 0 1, limit lower=-0.7 upper=0.7 effort=1.0 velocity=0.005
- added joint head_upperlegM2_yaw_joint: type revolute, parent head_link, child upperleg_M2_yaw_link, origin xyz=0.02165 -0.0125 -0.008 rpy=0 0 0, axis 0 0 1, limit lower=-0.7 upper=0.7 effort=1.0 velocity=0.005
- added joint head_upperlegM3_yaw_joint: type revolute, parent head_link, child upperleg_M3_yaw_link, origin xyz=0 0.025 -0.008 rpy=0 0 0, axis 0 0 1, limit lower=-0.7 upper=0.7 effort=1.0 velocity=0.005
- joint basefoot_peg_M1_basefoot_peg_M1_joint_joint: axis (none) -> 0 0 1; limit (none) -> lower=0.0 upper=0.05 effort=100000.0 velocity=50.0; type fixed -> prismatic
- joint basefoot_peg_M2_basefoot_peg_M2_joint_joint: axis (none) -> 0 0 1; limit (none) -> lower=0.0 upper=0.05 effort=100000.0 velocity=50.0; type fixed -> prismatic
- joint basefoot_peg_M3_basefoot_peg_M3_joint_joint: axis (none) -> 0 0 1; limit (none) -> lower=0.0 upper=0.05 effort=100000.0 velocity=50.0; type fixed -> prismatic
- joint head_upperlegM1_joint: origin xyz=-0.02165 -0.0125 -0.008 rpy=3.14159 0 0.523599 -> xyz=0 0 0 rpy=3.14159 0 0.523599; parent head_link -> upperleg_M1_yaw_link
- joint head_upperlegM2_joint: origin xyz=0.02165 -0.0125 -0.008 rpy=3.14159 0 2.61799 -> xyz=0 0 0 rpy=3.14159 0 2.61799; parent head_link -> upperleg_M2_yaw_link
- joint head_upperlegM3_joint: origin xyz=0 0.025 -0.008 rpy=3.14159 0 -1.5708 -> xyz=0 0 0 rpy=3.14159 0 -1.5708; parent head_link -> upperleg_M3_yaw_link
